File: Kicad-all-band-amp-April-2026/all-band-amp-April-2026/all-band-amp-April-2026.kicad_pcb (KiCad board)
At the start: 2 copper layers, 139.5 x 101 mm, 128 parts, among them J1 SWR1, J10 Aux In, J11 LPF, J12 Digi In/Out, J13 12v/5v Outputs, J14 TX2/RX2, J15 TX0/RX0, J16 50v In., J17 PWM Out, J18 PTT IN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

Commit message: change componet values
Parts:
- R43: value 1milli -> Shunt Not Fitted
- R44, R45: value 4k7 -> 1k5

Commit message: update functions
Parts:
- R3, R7: value 1k5 -> 1k5-3k3
