File: Kicad-all-band-amp-April-2026/all-band-amp-April-2026/all-band-amp-April-2026.kicad_pcb (KiCad board)
At the start: 2 copper layers, 139.5 x 101 mm, 128 parts, among them J1 SWR1, J10 Aux In, J11 LPF, J12 Digi In/Out, J13 12v/5v Outputs, J14 TX2/RX2, J15 TX0/RX0, J16 50v In., J17 PWM Out, J18 PTT IN, J19 DISPLAY POWER, J2 SWR2, J20 5V Output, J21 RS232, J22 UDPI, J23 12v Output, J24 12v Output, J25 Temp 2, J26 Power Link, J3 I opt Input, J4 RF In Level, J5 50v In., J6 Temp, J7 Conn_01x03_Pin, J8 12v Input, J9 I2c Output, Q1 2n2222, Q2 2n2222, SW1 SW_DIP_x02, U1 LTV-847, U2 MCP23017_SP, U3 LM393, U4 MIC2981/82YN, U5 MIC2981/82YN, U6 R-78E5.0-1.0, U7 MAX232N, U8 LTV-827, U9 ACS712xLCTR-30A

Commit message: change some values - alter boards
Parts:
- R24, R25: value 10k -> 4k7
Other:
- board text added: "1k5"

Commit message: update pcb's
Parts:
- added C26: 10nf, Capacitor_THT:C_Disc_D3.4mm_W2.1mm_P2.50mm, F.Cu at (146.0, 130.2)
- added J27: SWR trip out, Connector_JST:JST_EH_B2B-EH-A_1x02_P2.50mm_Vertical, F.Cu at (152.2, 140.0)
- added R46: 1k5, Resistor_THT:R_Axial_DIN0207_L6.3mm_D2.5mm_P7.62mm_Horizontal, F.Cu at (147.9, 135.2)
- added R47: 1k, Resistor_THT:R_Axial_DIN0207_L6.3mm_D2.5mm_P7.62mm_Horizontal, F.Cu at (149.2, 129.0)
Connections:
- net Net-(J13-Pin_3) renamed /SWR
Routing:
- net /SWR: track 59.0 -> 76.1 mm
- net Net-(J27-Pin_2): track 0.00 -> 14.9 mm
Other:
- board text added: "SWR trip"
