File: Kicad-all-band-amp-April-2026/all-band-amp-April-2026/all-band-amp-April-2026.kicad_pcb (KiCad board)
At the start: 2 copper layers, 139.5 x 101 mm, 132 parts, among them J1 SWR1, J10 Aux In, J11 LPF, J12 Digi In/Out, J13 12v/5v Outputs, J14 TX2/RX2, J15 TX0/RX0, J16 50v In., J17 PWM Out, J18 PTT IN, J19 DISPLAY POWER, J2 SWR2, J20 5V Output, J21 RS232, J22 UDPI, J23 12v Output, J24 12v Output, J25 Temp 2, J26 Power Link, J27 SWR trip out, J3 I opt Input, J4 RF In Level, J5 50v In., J6 Temp, J7 Conn_01x03_Pin, J8 12v Input, J9 I2c Output, Q1 2n2222, Q2 2n2222, SW1 SW_DIP_x02, U1 LTV-847, U2 MCP23017_SP, U3 LM393, U4 MIC2981/82YN, U5 MIC2981/82YN, U6 R-78E5.0-1.0, U7 MAX232N, U8 LTV-827, U9 ACS712xLCTR-30A

Commit message: update pcb's
Parts:
- removed J26: Power Link, my-footprints:AMASS_XT90-M_1x02_P11.00mm_Vertical
- added C27: 10nf, Capacitor_THT:C_Disc_D3.4mm_W2.1mm_P2.50mm, F.Cu at (105.9, 67.1)
- added C28: 100nf 2.5mm, Capacitor_THT:C_Disc_D3.4mm_W2.1mm_P2.50mm, F.Cu at (70.2, 108.3)
- added C29: 10nf, Capacitor_THT:C_Disc_D3.4mm_W2.1mm_P2.50mm, F.Cu at (104.4, 123.7)
- added C30: 10nf, Capacitor_THT:C_Disc_D3.4mm_W2.1mm_P2.50mm, F.Cu at (102.2, 116.8)
- added H5: 50v Ouput, my-footprints:PowerPad9mm, F.Cu at (66.5, 53.6)
- added H6: 50v Input, my-footprints:PowerPad9mm, F.Cu at (66.0, 63.8)
- added J28: SWR trip out, Connector_JST:JST_EH_B2B-EH-A_1x02_P2.50mm_Vertical, F.Cu at (64.0, 99.0)
- added J29: SWR trip out, Connector_JST:JST_EH_B2B-EH-A_1x02_P2.50mm_Vertical, F.Cu at (96.2, 47.5)
- added J30: SWR trip out, Connector_JST:JST_EH_B2B-EH-A_1x02_P2.50mm_Vertical, F.Cu at (129.9, 85.6)
- added J31: SWR trip out, Connector_JST:JST_EH_B2B-EH-A_1x02_P2.50mm_Vertical, F.Cu at (64.0, 124.0)
- added JP3: Jumper_2_Open, my-footprints:SolderJumper-2_P1.3mm_Open_TrianglePad1.0x1.5mm-mod, F.Cu at (136.2, 101.9)
- added JP4: Jumper_2_Open, my-footprints:SolderJumper-2_P1.3mm_Open_TrianglePad1.0x1.5mm-mod, F.Cu at (131.8, 101.9)
- added R48: 10k, Resistor_THT:R_Axial_DIN0207_L6.3mm_D2.5mm_P7.62mm_Horizontal, F.Cu at (71.9, 122.7)
- added R49: 10k, Resistor_THT:R_Axial_DIN0207_L6.3mm_D2.5mm_P7.62mm_Horizontal, F.Cu at (72.9, 107.3)
- added RV1: 10k, Potentiometer_THT:Potentiometer_Bourns_3296W_Vertical, F.Cu at (78.4, 127.3)
- added RV2: 10k, Potentiometer_THT:Potentiometer_Bourns_3296W_Vertical, F.Cu at (78.4, 133.1)
- added U10: LM358, Package_DIP:DIP-8_W7.62mm, F.Cu at (71.8, 118.7)
- C23: value 10uf -> 10uf-220uf
- J1: value SWR1 -> SWR
- J2: value SWR2 -> LPF
- Q2: value 2n2222 -> 2N7000; footprint Package_TO_SOT_THT:TO-92_HandSolder -> Package_TO_SOT_THT:TO-92_Inline
- R39, R41: value 220k -> 220k-1M
- R42: value 1k5 -> 10k
- R43: value Shunt Not Fitted -> Shunt I>30a
- R6: value 47k opt -> 47k/0r opt
- R8: value 680rr -> 680r
- moved D11 27.2 mm to (72.8, 104.1)
- moved C19 21.9 mm to (76.2, 97.2)
- moved R6 9.37 mm to (63.2, 79.6)
- moved J3 9.28 mm to (64.0, 87.8)
- moved D5 7.52 mm to (91.4, 136.9), turned to 180 degrees
- moved D4 6.53 mm to (98.2, 124.0), turned to -90 degrees
- moved C4 4.25 mm to (95.2, 124.0)
- moved D6 3.81 mm to (97.5, 52.8), turned to -90 degrees
- moved R46 3.61 mm to (149.1, 131.8)
- moved R11 2.95 mm to (94.7, 52.8), turned to -90 degrees
- moved C6 2.86 mm to (101.9, 54.4), turned to -90 degrees
- moved R10 2.66 mm to (91.3, 133.6)
- moved R9 2.46 mm to (83.7, 130.0)
- moved Q2 2.11 mm to (101.2, 60.4), turned to -90 degrees
- moved C5 1.69 mm to (95.4, 130.1), turned to -90 degrees
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Connections:
- net Net-(D8-K) renamed /SWR_OPT2
- A1 pad 21: unconnected-(A1-D26-Pad21) -> /D26
- C4 pad 1: /A3 -> Net-(D4-K)
- C5 pad 1: /A10 -> Net-(D5-K)
- D4 pad 1: /A3 -> Net-(D4-K)
- D5 pad 1: /A10 -> Net-(D5-K)
- Q2 pad 1: /IN8 -> GND
- Q2 pad 3: GND -> /IN8
- R10 pad 1: /A10 -> Net-(D5-K)
- R7 pad 2: /A3 -> Net-(D4-K)
- R8 pad 1: /A3 -> Net-(D4-K)
- R9 pad 2: /A10 -> Net-(D5-K)
Routing:
- net /D26: track 0.00 -> 47.0 mm
- net /SWR_OPT2: track 9.51 -> 53.3 mm
- net +5V: track 342.0 -> 382.5 mm, vias 2 -> 0
- net Net-(U10B--): track 0.00 -> 37.9 mm
- net Net-(D5-K): track 0.00 -> 37.5 mm
- net Net-(D11-K): track 32.9 -> 3.38 mm
- net Net-(D4-K): track 0.00 -> 27.3 mm
- net /A10: track 32.3 -> 54.1 mm
- net /712OUT: track 56.5 -> 74.2 mm
- net Net-(U10A--): track 0.00 -> 14.4 mm
- net Net-(D7-K): track 40.6 -> 54.3 mm
- net /IN8: track 73.1 -> 62.3 mm, vias 1 -> 0
- net /A3: track 47.8 -> 58.1 mm, vias 1 -> 0
- net VCC: track 191.8 -> 199.6 mm, vias 1 -> 0
- net /D11: track 0.00 -> 5.48 mm
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- added copper zone on In1.Cu, net GND
- added copper zone on In2.Cu, net GND
Other:
- copper layers 2 -> 4
- board text added: "+5v"
- board text added: "12v IN OUTS"
- board text added: "12v OUT"
- board text added: "AUX In Out"
- board text added: "I IN OUT"
- board text added: "INPUT"
- board text added: "LDMOS Controller v2.10d"
- board text added: "LPF"
- board text added: "OPT ERROR IN"
- board text added: "REV"
- board text added: "SCL"
- board text added: "SDA"
- board text added: "SWR Center Pin FWD"
- board text added: "SWR trip Opt"
- board text added: "SWR trip Opt1"
- board text added: "SWR trip Opt2"
- board text added: "Short JP4 & JP3 to use D7 & D8 as outputs R32 R33 DNF"
- board text added: "Spare 1"
- board text added: "Spare 2"
- board text added: "Thinary Nano 4808 MEGACOREX CODE https://github.com/MCUdude/MegaCoreX"
- board text removed: "12v IN"
- board text removed: "12v OUTPUTS"
- board text removed: "AUX In"
- board text removed: "ERROR IN"
- board text removed: "SCL SDA"
- board text removed: "SWR trip"
- board text removed: "SWR1 Center Pin FWD"
- board text removed: "SWR2 Center Pin FWD"
- board text removed: "Thinary Nano 4808 MEGACOREX CODE"
