File: Kicad-all-band-amp-April-2026/all-band-amp-April-2026/all-band-amp-April-2026.kicad_sch (KiCad schematic)
At the start: 124 parts, among them J1 SWR1, J10 Aux In, J11 LPF, J12 Digi In/Out, J13 12v/5v Outputs, J14 TX2/RX2, J15 TX0/RX0, J16 50v In., J17 PWM Out, J18 PTT IN, J19 DISPLAY POWER, J2 SWR2, J20 5V Output, J22 UDPI, J23 12v Output, J24 12v Output, J25 Temp 2, J26 Power Link, J27 SWR trip out, J3 I opt Input, J4 RF In Level, J5 50v In., J6 Temp, J7 Conn_01x03_Pin, J8 12v Input, J9 I2c Output, Q1 2n2222, Q2 2n2222, U1 LTV-847, U2 MCP23017_SP, U3 LM393, U4 MIC2981/82YN, U5 MIC2981/82YN, U6 R-78E5.0-1.0, U8 LTV-827, U9 ACS712xLCTR-30A

Commit message: update pcb's
Parts:
- removed J26: Power Link, my-footprints:AMASS_XT90-M_1x02_P11.00mm_Vertical, symbol Connector:Conn_01x02_Pin
- removed Q2: 2n2222, Package_TO_SOT_THT:TO-92_HandSolder, symbol Transistor_BJT:BC547
- added C27, C29, C30: 10nf, Capacitor_THT:C_Disc_D3.4mm_W2.1mm_P2.50mm, symbol Device:C
- added C28: 100nf 2.5mm, Capacitor_THT:C_Disc_D3.4mm_W2.1mm_P2.50mm, symbol Device:C
- added H5: 50v Ouput, my-footprints:PowerPad9mm, symbol Mechanical:MountingHole_Pad
- added H6: 50v Input, my-footprints:PowerPad9mm, symbol Mechanical:MountingHole_Pad
- added J28, J29, J30, J31: SWR trip out, Connector_JST:JST_EH_B2B-EH-A_1x02_P2.50mm_Vertical, symbol Connector:Conn_01x02_Pin
- added JP3, JP4: Jumper_2_Open, my-footprints:SolderJumper-2_P1.3mm_Open_TrianglePad1.0x1.5mm-mod, symbol Jumper:Jumper_2_Open
- added Q2: 2N7000, Package_TO_SOT_THT:TO-92_Inline, symbol Transistor_FET:2N7000
- added R48, R49: 10k, Resistor_THT:R_Axial_DIN0207_L6.3mm_D2.5mm_P7.62mm_Horizontal, symbol Device:R
- added RV1, RV2: 10k, Potentiometer_THT:Potentiometer_Bourns_3296W_Vertical, symbol Device:R_Potentiometer
- added U10: LM358, Package_DIP:DIP-8_W7.62mm, symbol Amplifier_Operational:LM358
- C23: value 10uf -> 10uf-220uf
- J1: value SWR1 -> SWR
- J2: value SWR2 -> LPF
- R39, R41: value 220k -> 220k-1M
- R42: value 1k5 -> 10k
- R43: value Shunt Not Fitted -> Shunt I>30a
- R6: value 47k opt -> 47k/0r opt
- R8: value 680rr -> 680r
Connections:
- net +5V: now also C28.1, U10.8 (V+)
- net 50V_: now also H5.1
- net 50v_In: now also H6.1
- net 712OUT: now also C27.1, J29.2 (Pin_2)
- net A10: now also C29.1, R49.1, U10.7; no longer C5.1, D5.1 (K), R10.1, R9.2
- net A3: now also C30.1, R48.1, U10.1; no longer C4.1, D4.1 (K), R7.2, R8.1
- net D11: now also J30.2 (Pin_2)
- net D7: now also JP4.1 (A)
- net D8: now also JP3.1 (A)
- net GND: now also C27.2, C28.2, C29.2, C30.2, J28.1 (Pin_1), J29.1 (Pin_1), J30.1 (Pin_1), J31.1 (Pin_1), Q2.1 (S), RV1.3, RV2.3, U10.4 (V-)
- net IN8: now also Q2.3 (D)
- net at C24.1, R42.2: now also Q2.2 (G)
- net at R29.2, U8.1: now also JP4.2 (B)
- net SWR_OPT2: now reaches D8.1 (K), D9.1 (K), R42.1
- net SWR_OPT2: now also J28.2 (Pin_2)
- net D26: now reaches A1.21 (D26)
- net D26: now also J31.2 (Pin_2)
- net at R28.2, U8.3: now also JP3.2 (B)
- new net: C5.1, D5.1 (K), R10.1, R9.2, U10.5 (+)
- new net: R49.2, RV2.1, RV2.2, U10.6 (-)
- new net: R48.2, RV1.1, RV1.2, U10.2 (-)
- new net: C4.1, D4.1 (K), R7.2, R8.1, U10.3 (+)
- no-connect marks 5 -> 3
Other:
- note added: "Current Sense Option"
- note added: "Note: To use D7/D8 as outputs dont fit LTV-827 And short pins 8-1 together and pins 6-3 tgether DNF R32 R33"
- note added: "Power 5v Display"
- note added: "SWR Opt. Trip out Protection Board etc."
- note added: "Spare In/Outs"
- note removed: "Current Sense"
- note removed: "Power"
- note removed: "SWR Trip out Protection Board etc."
- moved on the sheet: C26, C4, C5, C6, D4, D5, D6, J1, J12, J16, J17, J25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
