File: N-Con-Board-2026/N-Con-Board-2026.kicad_sch (KiCad schematic)
At the start: 22 parts, among them J1 SMA-AMP-In, J2 N-Type-Antenna, J3 Rig N-Type, J4 12v Bias Out, J5 AMP/LPF Output, J6 PTT, J7 12v Input, K1 G2RL-1-E-DC12, K2 G2RL-1-E-DC12, K3 HK4100F-DC12V-SHG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

Commit message: update pcb's
Other:
- moved on the sheet: H1, H2, H3, H4
Changed lines of the file:
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@@
 	)
 	(junction
-		(at 30.48 139.7)
+		(at 45.72 143.51)
 		(diameter 0)
 		(color 0 0 0 0)
 	)
 	(junction
-		(at 30.48 133.35)
+		(at 45.72 137.16)
 		(diameter 0)
 		(color 0 0 0 0)
@@
 	(wire
 		(pts
-			(xy 30.48 139.7) (xy 53.34 139.7)
+			(xy 45.72 143.51) (xy 68.58 143.51)
 		)
 		(stroke
@@
 	(wire
 		(pts
-			(xy 30.48 133.35) (xy 53.34 133.35)
+			(xy 45.72 137.16) (xy 68.58 137.16)
 		)
 		(stroke
@@
 	(wire
 		(pts
-			(xy 26.67 133.35) (xy 30.48 133.35)
+			(xy 41.91 137.16) (xy 45.72 137.16)
 		)
 		(stroke
@@
 	(symbol
 		(lib_id "power:GND")
-		(at 30.48 139.7 0)
+		(at 45.72 143.51 0)
 		(unit 1)
 		(body_style 1)
@@
 		(fields_autoplaced yes)
 		(property "Reference" "#PWR016"
-			(at 30.48 146.05 0)
+			(at 45.72 149.86 0)
 			(hide yes)
 			(show_name no)
@@
 		)
 		(property "Value" "GND"
-			(at 30.48 144.78 0)
+			(at 45.72 148.59 0)
 			(show_name no)
 			(do_not_autoplace no)
@@
 		)
 		(property "Footprint" ""
-			(at 30.48 139.7 0)
+			(at 45.72 143.51 0)
 			(hide yes)
 			(show_name no)
@@
 		)
 		(property "Datasheet" ""
-			(at 30.48 139.7 0)
+			(at 45.72 143.51 0)
 			(hide yes)
 			(show_name no)
@@
 		)
 		(property "Description" "Power symbol creates a global label with name \"GND\" , ground"
-			(at 30.48 139.7 0)
+			(at 45.72 143.51 0)
 			(hide yes)
 			(show_name no)
@@
 	(symbol
 		(lib_id "power:GND")
-		(at 26.67 133.35 0)
+		(at 41.91 137.16 0)
 		(unit 1)
 		(body_style 1)
@@
 		(fields_autoplaced yes)
 		(property "Reference" "#PWR017"
-			(at 26.67 139.7 0)
+			(at 41.91 143.51 0)
 			(hide yes)
 			(show_name no)
@@
 		)
 		(property "Value" "GND"
-			(at 26.67 138.43 0)
+			(at 41.91 142.24 0)
 			(show_name no)
 			(do_not_autoplace no)
@@
 		)
 		(property "Footprint" ""
-			(at 26.67 133.35 0)
+			(at 41.91 137.16 0)
 			(hide yes)
 			(show_name no)
@@
 		)
 		(property "Datasheet" ""
-			(at 26.67 133.35 0)
+			(at 41.91 137.16 0)
 			(hide yes)
 			(show_name no)
@@
 		)
 		(property "Description" "Power symbol creates a global label with name \"GND\" , ground"
-			(at 26.67 133.35 0)
+			(at 41.91 137.16 0)
 			(hide yes)
 			(show_name no)
@@
 	(symbol
 		(lib_id "Mechanical:MountingHole_Pad")
-		(at 53.34 137.16 0)
+		(at 68.58 140.97 0)
 		(unit 1)
 		(body_style 1)
@@
 		(fields_autoplaced yes)
 		(property "Reference" "H4"
-			(at 55.88 134.6199 0)
+			(at 71.12 138.4299 0)
 			(show_name no)
 			(do_not_autoplace no)
@@
 		)
 		(property "Value" "MountingHole_Pad"
-			(at 55.88 137.1599 0)
+			(at 71.12 140.9699 0)
 			(show_name no)
 			(do_not_autoplace no)
@@
 		)
 		(property "Footprint" "MountingHole:MountingHole_3.5mm_Pad_Via"
-			(at 53.34 137.16 0)
+			(at 68.58 140.97 0)
 			(hide yes)
 			(show_name no)
@@
 		)
 		(property "Datasheet" ""
-			(at 53.34 137.16 0)
+			(at 68.58 140.97 0)
 			(hide yes)
 			(show_name no)
@@
 		)
 		(property "Description" "Mounting Hole with connection"
-			(at 53.34 137.16 0)
+			(at 68.58 140.97 0)
 			(hide yes)
 			(show_name no)
@@
 	(symbol
 		(lib_id "Mechanical:MountingHole_Pad")
-		(at 53.34 130.81 0)
+		(at 68.58 134.62 0)
 		(unit 1)
 		(body_style 1)
@@
 		(fields_autoplaced yes)
 		(property "Reference" "H3"
-			(at 55.88 128.2699 0)
+			(at 71.12 132.0799 0)
 			(show_name no)
 			(do_not_autoplace no)
@@
 		)
 		(property "Value" "MountingHole_Pad"
-			(at 55.88 130.8099 0)
+			(at 71.12 134.6199 0)
 			(show_name no)
 			(do_not_autoplace no)
@@
 		)
 		(property "Footprint" "MountingHole:MountingHole_3.5mm_Pad_Via"
-			(at 53.34 130.81 0)
+			(at 68.58 134.62 0)
 			(hide yes)
 			(show_name no)
@@
 		)
 		(property "Datasheet" ""
-			(at 53.34 130.81 0)
+			(at 68.58 134.62 0)
 			(hide yes)
 			(show_name no)
@@
 		)
 		(property "Description" "Mounting Hole with connection"
-			(at 53.34 130.81 0)
+			(at 68.58 134.62 0)
 			(hide yes)
 			(show_name no)
@@
 	(symbol
 		(lib_id "Mechanical:MountingHole_Pad")
-		(at 30.48 137.16 0)
+		(at 45.72 140.97 0)
 		(unit 1)
 		(body_style 1)
@@
 		(fields_autoplaced yes)
 		(property "Reference" "H2"
-			(at 33.02 134.6199 0)
+			(at 48.26 138.4299 0)
 			(show_name no)
 			(do_not_autoplace no)
@@
 		)
 		(property "Value" "MountingHole_Pad"
-			(at 33.02 137.1599 0)
+			(at 48.26 140.9699 0)
 			(show_name no)
 			(do_not_autoplace no)
@@
 		)
 		(property "Footprint" "MountingHole:MountingHole_3.5mm_Pad_Via"
-			(at 30.48 137.16 0)
+			(at 45.72 140.97 0)
 			(hide yes)
 			(show_name no)
@@
 		)
 		(property "Datasheet" ""
-			(at 30.48 137.16 0)
+			(at 45.72 140.97 0)
 			(hide yes)
 			(show_name no)
@@
 		)
 		(property "Description" "Mounting Hole with connection"
-			(at 30.48 137.16 0)
+			(at 45.72 140.97 0)
 			(hide yes)
 			(show_name no)
@@
 	(symbol
 		(lib_id "Mechanical:MountingHole_Pad")
-		(at 30.48 130.81 0)
+		(at 45.72 134.62 0)
 		(unit 1)
 		(body_style 1)
@@
 		(fields_autoplaced yes)
 		(property "Reference" "H1"
-			(at 33.02 128.2699 0)
+			(at 48.26 132.0799 0)
 			(show_name no)
 			(do_not_autoplace no)
@@
 		)
 		(property "Value" "MountingHole_Pad"
-			(at 33.02 130.8099 0)
+			(at 48.26 134.6199 0)
 			(show_name no)
 			(do_not_autoplace no)
@@
 		)
 		(property "Footprint" "MountingHole:MountingHole_3.5mm_Pad_Via"
-			(at 30.48 130.81 0)
+			(at 45.72 134.62 0)
 			(hide yes)
 			(show_name no)
@@
 		)
 		(property "Datasheet" ""
-			(at 30.48 130.81 0)
+			(at 45.72 134.62 0)
 			(hide yes)
 			(show_name no)
@@
 		)
 		(property "Description" "Mounting Hole with connection"
-			(at 30.48 130.81 0)
+			(at 45.72 134.62 0)
 			(hide yes)
 			(show_name no)
