File: N-Con-Board-2026/N-Con-Board-2026.kicad_pcb (KiCad board)
At the start: 2 copper layers, 105 x 55 mm, 22 parts, among them J1 SMA-AMP-In, J2 N-Type-Antenna, J3 Rig N-Type, J4 12v Bias Out, J5 AMP/LPF Output, J6 PTT, J7 12v Input, K1 G2RL-1-E-DC12, K2 G2RL-1-E-DC12, K3 HK4100F-DC12V-SHG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

Commit message: change some values - alter boards
Parts:
- J5: value AMP/LPF Output -> From AMP/LPF Output
Other:
- board text added: "N-Type Board Rev.2c"
- board text removed: "N-Type Board Rev.2b"
