File: N-Con-Board-2026/N-Con-Board-2026.kicad_pcb (KiCad board)
At the start: 2 copper layers, 105 x 55 mm, 22 parts, among them J1 SMA-AMP-In, J2 N-Type-Antenna, J3 Rig N-Type, J4 12v Bias Out, J5 From AMP/LPF Output, J6 PTT, J7 12v Input, K1 G2RL-1-E-DC12, K2 G2RL-1-E-DC12, K3 HK4100F-DC12V-SHG, SW1 SW_Push_Test

Commit message: update pcb's
Parts:
- J5: value From AMP/LPF Output -> AMP/LPF Output
- moved C2 11.3 mm to (91.6, 62.6)
- moved K3 3.06 mm to (95.5, 67.8)
- moved J4 1.98 mm to (115.6, 76.2), turned to 0 degrees
- moved R1 0.84 mm to (152.9, 75.1)
Routing:
- net +12V: track 46.4 -> 40.8 mm
- net Net-(D2-A): track 75.0 -> 71.4 mm
- net Net-(D1-K): track 74.6 -> 77.1 mm
Other:
- board text added: "N-Type Board Rev.2d"
- board text removed: "N-Type Board Rev.2c"
