File: RFA-Board-2026/RFA-Board-2026/RFA-Board-2026.kicad_pcb (KiCad board)
At the start: 2 copper layers, 68.2 x 39.5 mm, 18 parts, among them J1 SMA Connector, J2 SMA Connector, J3 Conn_01x02_Pin, J4 Conn_01x02_Pin, K1 IM26GR, U1 RFA-10DB

Commit message: update pcb files to kicad 10
Parts:
- J1, J2: footprint Connector_Coaxial:SMA_Molex_73251-2200_Horizontal_MOD -> RFA:SMA_Molex_73251-2200_Horizontal_MOD

Commit message: update pcb's
Parts:
- C1, C2: footprint Capacitor_SMD:C_1206_3216Metric_Pad1.33x1.80mm_HandSolder -> RFA:C_1206_3216Metric_Pad1.33x1.80mm_HandSolder-mod
- D1, D2: footprint Diode_SMD:D_MELF-RM10_Universal_Handsoldering -> RFA:D_MELF-RM10_Universal_Handsoldering-mod
- R1, R2, R3, R4: footprint Resistor_SMD:R_1206_3216Metric_Pad1.30x1.75mm_HandSolder -> RFA:R_1206_3216Metric_Pad1.30x1.75mm_HandSolder-mod
- moved H1 0.14 mm to (123.6, 87.0)
Changed lines of the file:
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@@
 		(embedded_fonts no)
 	)
-	(footprint "Resistor_SMD:R_1206_3216Metric_Pad1.30x1.75mm_HandSolder"
+	(footprint "RFA:R_1206_3216Metric_Pad1.30x1.75mm_HandSolder-mod"
 		(layer "F.Cu")
 		(at 134.404 77.5)
@@
 		(tags "resistor handsolder")
 		(property "Reference" "R1"
-			(at 0.05 2.5 0)
+			(at -0.05 2 180)
 			(layer "F.SilkS")
 			(effects
@@
 		)
 		(property "Value" "3k3"
-			(at -2.95 3 0)
+			(at 1.95 3 180)
 			(layer "F.Fab")
 			(effects
@@
 		)
 		(property "Datasheet" ""
-			(at 0 0 0)
+			(at 0 0 180)
 			(layer "F.Fab")
 			(hide yes)
@@
 		)
 		(property "Description" "Resistor"
-			(at 0 0 0)
+			(at 0 0 180)
 			(layer "F.Fab")
 			(hide yes)
@@
 		)
 		(fp_text user "${REFERENCE}"
-			(at 0 0 0)
+			(at 0 0 180)
 			(layer "F.Fab")
 			(effects
@@
 		)
 	)
-	(footprint "Resistor_SMD:R_1206_3216Metric_Pad1.30x1.75mm_HandSolder"
+	(footprint "RFA:R_1206_3216Metric_Pad1.30x1.75mm_HandSolder-mod"
 		(layer "F.Cu")
 		(at 147.904 73)
@@
 		(tags "resistor handsolder")
 		(property "Reference" "R4"
-			(at 0 2 0)
+			(at -0.05 2 180)
 			(layer "F.SilkS")
 			(effects
@@
 		)
 		(property "Value" "1k5 or Not Fitted"
-			(at 3.05 -2.5 0)
+			(at 1.95 3 180)
 			(layer "F.Fab")
 			(effects
@@
 		)
 		(property "Datasheet" ""
-			(at 0 0 0)
+			(at 0 0 180)
 			(layer "F.Fab")
 			(hide yes)
@@
 		)
 		(property "Description" "Resistor"
-			(at 0 0 0)
+			(at 0 0 180)
 			(layer "F.Fab")
 			(hide yes)
@@
 		)
 		(fp_text user "${REFERENCE}"
-			(at 0 0 0)
+			(at 0 0 180)
 			(layer "F.Fab")
 			(effects
@@
 		)
 	)
-	(footprint "Diode_SMD:D_MELF-RM10_Universal_Handsoldering"
+	(footprint "RFA:D_MELF-RM10_Universal_Handsoldering-mod"
 		(layer "F.Cu")
 		(at 144.954 77.5)
@@
 	(footprint "MountingHole:MountingHole_3.5mm_Pad_Via"
 		(layer "F.Cu")
-		(at 123.625 87.143845)
+		(at 123.625 87)
 		(descr "Mounting Hole 3.5mm, generated by kicad-footprint-generator mountinghole.py")
 		(tags "mountinghole")
@@
 				(font
 					(size 1.27 1.27)
-					(thickness 0.15)
 				)
 			)
@@
 				(font
 					(size 1.27 1.27)
+				)
+			)
+		)
+		(property "KiLib_Generator" "mounting_hardware/mounting_hole"
+			(at 0 0 0)
+			(layer "F.SilkS")
+			(hide yes)
+			(effects
+				(font
+					(size 1 1)
 					(thickness 0.15)
 				)
@@
 			(pintype "input")
 			(zone_connect 2)
-			(teardrops
-				(best_length_ratio 0.5)
-				(max_length 1)
-				(best_width_ratio 1)
-				(max_width 2)
-				(curved_edges no)
-				(filter_ratio 0.9)
-				(enabled yes)
-				(allow_two_segments yes)
-				(prefer_zone_connections yes)
-			)
 		)
 		(pad "1" thru_hole circle
@@
 			(pintype "input")
 			(zone_connect 2)
-			(teardrops
-				(best_length_ratio 0.5)
-				(max_length 1)
-				(best_width_ratio 1)
-				(max_width 2)
-				(curved_edges no)
-				(filter_ratio 0.9)
-				(enabled yes)
-				(allow_two_segments yes)
-				(prefer_zone_connections yes)
-			)
 		)
 		(pad "1" thru_hole circle
@@
 			(pintype "input")
 			(zone_connect 2)
-			(teardrops
-				(best_length_ratio 0.5)
-				(max_length 1)
-				(best_width_ratio 1)
-				(max_width 2)
-				(curved_edges no)
-				(filter_ratio 0.9)
-				(enabled yes)
-				(allow_two_segments yes)
-				(prefer_zone_connections yes)
-			)
 		)
 		(pad "1" thru_hole circle
@@
 			(pintype "input")
 			(zone_connect 2)
-			(teardrops
-				(best_length_ratio 0.5)
-				(max_length 1)
-				(best_width_ratio 1)
-				(max_width 2)
-				(curved_edges no)
-				(filter_ratio 0.9)
-				(enabled yes)
-				(allow_two_segments yes)
-				(prefer_zone_connections yes)
-			)
 		)
 		(pad "1" thru_hole circle
-			(at 0 -0.143845)
+			(at 0 0)
 			(size 7 7)
 			(drill 3.5)
@@
 			(pintype "input")
 			(zone_connect 2)
-			(teardrops
-				(best_length_ratio 0.5)
-				(max_length 1)
-				(best_width_ratio 1)
-				(max_width 2)
-				(curved_edges no)
-				(filter_ratio 0.9)
-				(enabled yes)
-				(allow_two_segments yes)
-				(prefer_zone_connections yes)
-			)
 		)
 		(pad "1" thru_hole circle
@@
 			(pintype "input")
 			(zone_connect 2)
-			(teardrops
-				(best_length_ratio 0.5)
-				(max_length 1)
-				(best_width_ratio 1)
-				(max_width 2)
-				(curved_edges no)
-				(filter_ratio 0.9)
-				(enabled yes)
-				(allow_two_segments yes)
-				(prefer_zone_connections yes)
-			)
 		)
 		(pad "1" thru_hole circle
@@
 			(pintype "input")
 			(zone_connect 2)
-			(teardrops
-				(best_length_ratio 0.5)
-				(max_length 1)
-				(best_width_ratio 1)
-				(max_width 2)
-				(curved_edges no)
-				(filter_ratio 0.9)
-				(enabled yes)
-				(allow_two_segments yes)
-				(prefer_zone_connections yes)
-			)
 		)
 		(pad "1" thru_hole circle
@@
 			(pintype "input")
 			(zone_connect 2)
-			(teardrops
-				(best_length_ratio 0.5)
-				(max_length 1)
-				(best_width_ratio 1)
-				(max_width 2)
-				(curved_edges no)
-				(filter_ratio 0.9)
-				(enabled yes)
-				(allow_two_segments yes)
-				(prefer_zone_connections yes)
-			)
 		)
 		(pad "1" thru_hole circle
@@
 			(pintype "input")
 			(zone_connect 2)
-			(teardrops
-				(best_length_ratio 0.5)
-				(max_length 1)
-				(best_width_ratio 1)
-				(max_width 2)
-				(curved_edges no)
-				(filter_ratio 0.9)
-				(enabled yes)
-				(allow_two_segments yes)
-				(prefer_zone_connections yes)
-			)
 		)
 		(embedded_fonts no)
 	)
-	(footprint "Capacitor_SMD:C_1206_3216Metric_Pad1.33x1.80mm_HandSolder"
+	(footprint "RFA:C_1206_3216Metric_Pad1.33x1.80mm_HandSolder-mod"
 		(layer "F.Cu")
 		(at 127.8915 73)
@@
 		)
 	)
-	(footprint "Resistor_SMD:R_1206_3216Metric_Pad1.30x1.75mm_HandSolder"
+	(footprint "RFA:R_1206_3216Metric_Pad1.30x1.75mm_HandSolder-mod"
 		(layer "F.Cu")
 		(at 134.404 73)
@@
 		(tags "resistor handsolder")
 		(property "Reference" "R2"
-			(at 0.05 2 0)
+			(at -0.05 2 180)
 			(layer "F.SilkS")
 			(effects
@@
 		)
 		(property "Value" "560r"
-			(at 0.55 -2.5 0)
+			(at 1.95 3 180)
 			(layer "F.Fab")
 			(effects
@@
 		)
 		(property "Datasheet" ""
-			(at 0 0 0)
+			(at 0 0 180)
 			(layer "F.Fab")
 			(hide yes)
@@
 		)
 		(property "Description" "Resistor"
-			(at 0 0 0)
+			(at 0 0 180)
 			(layer "F.Fab")
 			(hide yes)
@@
 		)
 		(fp_text user "${REFERENCE}"
-			(at 0 0 0)
+			(at 0 0 180)
 			(layer "F.Fab")
 			(effects
@@
 		)
 	)
-	(footprint "Resistor_SMD:R_1206_3216Metric_Pad1.30x1.75mm_HandSolder"
+	(footprint "RFA:R_1206_3216Metric_Pad1.30x1.75mm_HandSolder-mod"
 		(layer "F.Cu")
 		(at 140.904 73 180)
@@
 		)
 	)
-	(footprint "Capacitor_SMD:C_1206_3216Metric_Pad1.33x1.80mm_HandSolder"
+	(footprint "RFA:C_1206_3216Metric_Pad1.33x1.80mm_HandSolder-mod"
 		(layer "F.Cu")
 		(at 127.8915 77.5)
@@
 		)
 		(property "Value" "1nf"
-			(at 0 1.85 0)
+			(at -5.4375 2 0)
 			(layer "F.Fab")
 			(effects
@@
 		(embedded_fonts no)
 	)
-	(footprint "Diode_SMD:D_MELF-RM10_Universal_Handsoldering"
+	(footprint "RFA:D_MELF-RM10_Universal_Handsoldering-mod"
 		(layer "F.Cu")
 		(at 166.8 76.374 90)
@@
 		(tags "Diode Universal MELF RM10 Handsoldering SMD Thruhole ")
 		(property "Reference" "D2"
-			(at 0 -2.5 90)
+			(at 0 3 90)
 			(layer "F.SilkS")
 			(effects
@@
 		)
 		(property "Value" "BAT85"
-			(at 0 2.5 90)
+			(at 4 3 90)
 			(layer "F.Fab")
 			(effects
@@
 		(duplicate_pad_numbers_are_jumpers no)
 		(fp_line
-			(start 3.9 -1.61)
+			(start 6.3 -1.61)
 			(end -6.41 -1.61)
 			(stroke
@@
 		)
 		(fp_line
-			(start -6.41 -1.61)
-			(end -6.41 1.61)
-			(stroke
-				(width 0.12)
-				(type solid)
-			)
-			(layer "F.SilkS")
-		)
-		(fp_line
 			(start -6.41 1.61)
-			(end 3.9 1.61)
+			(end 6.4 1.61)
 			(stroke
 				(width 0.12)
@@
 		(pad "1" smd roundrect
 			(at -5 0 90)
-			(size 4.5 2.7)
+			(size 5 2.7)
 			(drill
 				(offset 1.1 0)
@@
 		(pad "2" smd roundrect
 			(at 5 0 270)
-			(size 4.5 2.7)
+			(size 5 2.7)
 			(drill
 				(offset 1.1 0)
@@
 		(layer "F.Cu")
 		(hatch none 0.1)
-		(priority 30017)
+		(priority 30018)
 		(attr
 			(teardrop
@@
 		(layer "F.Cu")
 		(hatch none 0.1)
-		(priority 30011)
+		(priority 30012)
 		(attr
 			(teardrop
@@
 		(layer "F.Cu")
 		(hatch none 0.1)
-		(priority 30023)
+		(priority 30024)
 		(attr
 			(teardrop
@@
 		(layer "F.Cu")
 		(hatch none 0.1)
-		(priority 30026)
+		(priority 30022)
 		(attr
 			(teardrop
@@
 		(layer "F.Cu")
 		(hatch none 0.1)
-		(priority 30022)
+		(priority 30023)
 		(attr
 			(teardrop
@@
 		(layer "F.Cu")
 		(hatch none 0.1)
-		(priority 30012)
+		(priority 30011)
 		(attr
 			(teardrop
@@
 		(polygon
 			(pts
-				(xy 166.65 83.524) (xy 166.95 83.524) (xy 167.8 82.524) (xy 166.8 81.173) (xy 165.8 82.524)
+				(xy 166.65 83.774) (xy 166.95 83.774) (xy 167.8 82.774) (xy 166.8 81.373) (xy 165.8 82.774)
 			)
 		)
@@
 		(layer "F.Cu")
 		(hatch none 0.1)
-		(priority 30018)
+		(priority 30017)
 		(attr
 			(teardrop
@@
 		(layer "F.Cu")
 		(hatch none 0.1)
-		(priority 30024)
+		(priority 30026)
 		(attr
 			(teardrop
@@
 		(fill yes
 			(thermal_gap 0.5)
-			(thermal_bridge_width 0.5)
+			(thermal_bridge_width 1)
 			(island_removal_mode 0)
 		)
