File: RFA-Board-2026/RFA-Board-2026/RFA-Board-2026.kicad_sch (KiCad schematic)
At the start: 18 parts, among them J1 SMA Connector, J2 SMA Connector, J3 Conn_01x02_Pin, J4 Conn_01x02_Pin, K1 IM26GR, U1 RFA-10DB

Commit message: update pcb files to kicad 10
Parts:
- J1, J2: footprint Connector_Coaxial:SMA_Molex_73251-2200_Horizontal_MOD -> RFA:SMA_Molex_73251-2200_Horizontal_MOD

Commit message: update pcb's
Parts:
- C1, C2: footprint Capacitor_SMD:C_1206_3216Metric_Pad1.33x1.80mm_HandSolder -> RFA:C_1206_3216Metric_Pad1.33x1.80mm_HandSolder-mod
- D1, D2: footprint Diode_SMD:D_MELF-RM10_Universal_Handsoldering -> RFA:D_MELF-RM10_Universal_Handsoldering-mod
- R1, R2, R3, R4: footprint Resistor_SMD:R_1206_3216Metric_Pad1.30x1.75mm_HandSolder -> RFA:R_1206_3216Metric_Pad1.30x1.75mm_HandSolder-mod
Changed lines of the file:
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@@
 			)
 		)
-		(property "Footprint" "Resistor_SMD:R_1206_3216Metric_Pad1.30x1.75mm_HandSolder"
+		(property "Footprint" "RFA:R_1206_3216Metric_Pad1.30x1.75mm_HandSolder-mod"
 			(at 138.938 90.17 90)
 			(hide yes)
@@
 			)
 		)
-		(property "Footprint" "Resistor_SMD:R_1206_3216Metric_Pad1.30x1.75mm_HandSolder"
+		(property "Footprint" "RFA:R_1206_3216Metric_Pad1.30x1.75mm_HandSolder-mod"
 			(at 121.412 100.33 90)
 			(hide yes)
@@
 			)
 		)
-		(property "Footprint" "Diode_SMD:D_MELF-RM10_Universal_Handsoldering"
+		(property "Footprint" "RFA:D_MELF-RM10_Universal_Handsoldering-mod"
 			(at 169.545 120.65 0)
 			(hide yes)
@@
 			)
 		)
-		(property "Footprint" "Diode_SMD:D_MELF-RM10_Universal_Handsoldering"
+		(property "Footprint" "RFA:D_MELF-RM10_Universal_Handsoldering-mod"
 			(at 118.745 109.22 0)
 			(hide yes)
@@
 			)
 		)
-		(property "Footprint" "Resistor_SMD:R_1206_3216Metric_Pad1.30x1.75mm_HandSolder"
+		(property "Footprint" "RFA:R_1206_3216Metric_Pad1.30x1.75mm_HandSolder-mod"
 			(at 127 84.582 90)
 			(hide yes)
@@
 			)
 		)
-		(property "Footprint" "Resistor_SMD:R_1206_3216Metric_Pad1.30x1.75mm_HandSolder"
+		(property "Footprint" "RFA:R_1206_3216Metric_Pad1.30x1.75mm_HandSolder-mod"
 			(at 124.968 92.71 90)
 			(hide yes)
@@
 			)
 		)
-		(property "Footprint" "Capacitor_SMD:C_1206_3216Metric_Pad1.33x1.80mm_HandSolder"
+		(property "Footprint" "RFA:C_1206_3216Metric_Pad1.33x1.80mm_HandSolder-mod"
 			(at 123.19 95.5548 0)
 			(hide yes)
@@
 			)
 		)
-		(property "Footprint" "Capacitor_SMD:C_1206_3216Metric_Pad1.33x1.80mm_HandSolder"
+		(property "Footprint" "RFA:C_1206_3216Metric_Pad1.33x1.80mm_HandSolder-mod"
 			(at 123.19 87.9348 0)
 			(hide yes)
