File: RFA_Board/RFA_Board.kicad_pcb (KiCad board)
At the start: 2 copper layers, 52 x 39.5 mm, 13 parts, among them J1 SMA Connector, J2 SMA Connector, J3 Conn_01x02_Pin, U1 RFA-10DB

Commit message: update pcb's
Parts:
- C1, C2: footprint Capacitor_SMD:C_1206_3216Metric_Pad1.33x1.80mm_HandSolder -> RFA:C_1206_3216Metric_Pad1.33x1.80mm_HandSolder-mod
- D1: footprint Diode_SMD:D_MELF-RM10_Universal_Handsoldering -> RFA:D_MELF-RM10_Universal_Handsoldering-mod
- J1, J2: footprint Connector_Coaxial:SMA_Molex_73251-2200_Horizontal_MOD -> RFA:SMA_Molex_73251-2200_Horizontal_MOD
- J3: footprint solderwire:SolderWirePad_1x02_SMD_5x8mm -> RFA:SolderWirePad_1x02_SMD_12.5x8mm
- R1, R2, R3, R4: footprint Resistor_SMD:R_1206_3216Metric_Pad1.30x1.75mm_HandSolder -> RFA:R_1206_3216Metric_Pad1.30x1.75mm_HandSolder-mod
